Commit message: Lower initial pose, match kp and kd to puppersim for Pupper

File: resources/robots/pupper/pupper_v2a.urdf (robot description, URDF)
Before this commit: robot pupper_v2_dji, 17 links, 16 joints
Joints:
- joint leftFrontLegMotor: limit lower=-0.7854 upper=0.7854 effort=10 velocity=10 -> lower=-0.7854 upper=0.7854 effort=1.7 velocity=10
- joint leftFrontLowerLegMotor: limit lower=-2.87979 upper=2.87979 effort=10 velocity=10 -> lower=-2.87979 upper=2.87979 effort=1.7 velocity=10
- joint leftFrontUpperLegMotor: limit lower=-1.309 upper=4.45059 effort=10 velocity=10 -> lower=-1.309 upper=4.45059 effort=1.7 velocity=10
- joint leftRearLegMotor: limit lower=-0.7854 upper=0.7854 effort=10 velocity=10 -> lower=-0.7854 upper=0.7854 effort=1.7 velocity=10
- joint leftRearLowerLegMotor: limit lower=-2.87979 upper=2.87979 effort=10 velocity=10 -> lower=-2.87979 upper=2.87979 effort=1.7 velocity=10
- joint leftRearUpperLegMotor: limit lower=-1.309 upper=4.45059 effort=10 velocity=10 -> lower=-1.309 upper=4.45059 effort=1.7 velocity=10
- joint rightFrontLegMotor: limit lower=-0.7854 upper=0.7854 effort=10 velocity=10 -> lower=-0.7854 upper=0.7854 effort=1.7 velocity=10
- joint rightFrontLowerLegMotor: limit lower=-2.87979 upper=2.87979 effort=10 velocity=10 -> lower=-2.87979 upper=2.87979 effort=1.7 velocity=10
- joint rightFrontUpperLegMotor: limit lower=-1.309 upper=4.45059 effort=10 velocity=10 -> lower=-1.309 upper=4.45059 effort=1.7 velocity=10
- joint rightRearLegMotor: limit lower=-0.7854 upper=0.7854 effort=10 velocity=10 -> lower=-0.7854 upper=0.7854 effort=1.7 velocity=10
- joint rightRearLowerLegMotor: limit lower=-2.87979 upper=2.87979 effort=10 velocity=10 -> lower=-2.87979 upper=2.87979 effort=1.7 velocity=10
- joint rightRearUpperLegMotor: limit lower=-1.309 upper=4.45059 effort=10 velocity=10 -> lower=-1.309 upper=4.45059 effort=1.7 velocity=10

Commit message: reward tuning

File: resources/robots/pupper/pupper_v2a.urdf (robot description, URDF)
Before this commit: robot pupper_v2_dji, 17 links, 16 joints
Joints:
- joint leftFrontLowerLegMotor: limit lower=-2.87979 upper=2.87979 effort=1.7 velocity=10 -> lower=-2.87979 upper=0 effort=1.7 velocity=10
- joint leftRearLowerLegMotor: limit lower=-2.87979 upper=2.87979 effort=1.7 velocity=10 -> lower=-2.87979 upper=0 effort=1.7 velocity=10
- joint rightFrontLowerLegMotor: limit lower=-2.87979 upper=2.87979 effort=1.7 velocity=10 -> lower=-2.87979 upper=0.0 effort=1.7 velocity=10
- joint rightRearLowerLegMotor: limit lower=-2.87979 upper=2.87979 effort=1.7 velocity=10 -> lower=-2.87979 upper=0 effort=1.7 velocity=10

Commit message: update obs space, leg order for pupper

File: resources/robots/pupper/pupper_v2a.urdf (robot description, URDF)
Before this commit: robot pupper_v2_dji, 17 links, 16 joints
Joints:
- removed joint leftFrontLegMotor
- removed joint leftRearLegMotor
- removed joint rightFrontLegMotor
- removed joint rightRearLegMotor
- added joint leg1_rightFrontLegMotor: type revolute, parent pupper_v2_dji_chassis, child rightFrontLeg, origin xyz=-0.047 -0.103 0 rpy=0 0 -3.14159, axis 0 1.0 0, limit lower=-0.7854 upper=0.7854 effort=1.7 velocity=10
- added joint leg2_leftFrontLegMotor: type revolute, parent pupper_v2_dji_chassis, child leftFrontLeg, origin xyz=0.047 -0.1015 0 rpy=0 0 0, axis 0 -1.0 0, limit lower=-0.7854 upper=0.7854 effort=1.7 velocity=10
- added joint leg3_rightRearLegMotor: type revolute, parent pupper_v2_dji_chassis, child rightRearLeg, origin xyz=-0.047 0.097 0 rpy=0 0 -3.14159, axis 0 1.0 0, limit lower=-0.7854 upper=0.7854 effort=1.7 velocity=10
- added joint leg4_leftRearLegMotor: type revolute, parent pupper_v2_dji_chassis, child leftRearLeg, origin xyz=0.047 0.0985 0 rpy=0 0 0, axis 0 -1.0 0, limit lower=-0.7854 upper=0.7854 effort=1.7 velocity=10

Commit message: adjust sim paramters and reward for pupper

File: resources/robots/pupper/pupper_v2a.urdf (robot description, URDF)
Before this commit: robot pupper_v2_dji, 17 links, 16 joints
Joints:
- joint leftFrontLowerLegMotor: limit lower=-2.87979 upper=0 effort=1.7 velocity=10 -> lower=-2.87979 upper=0 effort=2 velocity=10
- joint leftFrontUpperLegMotor: limit lower=-1.309 upper=4.45059 effort=1.7 velocity=10 -> lower=-1.309 upper=4.45059 effort=2 velocity=10
- joint leftRearLowerLegMotor: limit lower=-2.87979 upper=0 effort=1.7 velocity=10 -> lower=-2.87979 upper=0 effort=2 velocity=10
- joint leftRearUpperLegMotor: limit lower=-1.309 upper=4.45059 effort=1.7 velocity=10 -> lower=-1.309 upper=4.45059 effort=2 velocity=10
- joint leg1_rightFrontLegMotor: limit lower=-0.7854 upper=0.7854 effort=1.7 velocity=10 -> lower=-0.7854 upper=0.7854 effort=2 velocity=10
- joint leg2_leftFrontLegMotor: limit lower=-0.7854 upper=0.7854 effort=1.7 velocity=10 -> lower=-0.7854 upper=0.7854 effort=2 velocity=10
- joint leg3_rightRearLegMotor: limit lower=-0.7854 upper=0.7854 effort=1.7 velocity=10 -> lower=-0.7854 upper=0.7854 effort=2 velocity=10
- joint leg4_leftRearLegMotor: limit lower=-0.7854 upper=0.7854 effort=1.7 velocity=10 -> lower=-0.7854 upper=0.7854 effort=2 velocity=10
- joint rightFrontLowerLegMotor: limit lower=-2.87979 upper=0.0 effort=1.7 velocity=10 -> lower=-2.87979 upper=0.0 effort=2 velocity=10
- joint rightFrontUpperLegMotor: limit lower=-1.309 upper=4.45059 effort=1.7 velocity=10 -> lower=-1.309 upper=4.45059 effort=2 velocity=10
- joint rightRearLowerLegMotor: limit lower=-2.87979 upper=0 effort=1.7 velocity=10 -> lower=-2.87979 upper=0 effort=2 velocity=10
- joint rightRearUpperLegMotor: limit lower=-1.309 upper=4.45059 effort=1.7 velocity=10 -> lower=-1.309 upper=4.45059 effort=2 velocity=10
